File: StreamLite.kicad_sch (KiCad schematic)
At the start: 54 parts, among them J1 Screw_Terminal_01x02, J2 Screw_Terminal_01x03, J3 Conn_01x06_Socket, J4 Screw_Terminal_01x03, J5 Screw_Terminal_01x03, J6 Screw_Terminal_01x03, J7 Screw_Terminal_01x03, Q1 BC327, Q10 BC327, Q11 BC337, Q12 NMOS, Q2 BC337, Q3 NMOS, Q4 BC327, Q5 BC337, Q6 NMOS, Q7 BC327, Q8 BC337, Q9 NMOS, SW1 Reset, U2 ESP32-WROOM-32, U3 AMS1117-3.3

Commit message: add parts
Parts:
- removed J1: Screw_Terminal_01x02, TerminalBlock_Phoenix:TerminalBlock_Phoenix_MPT-0,5-2-2.54_1x02_P2.54mm_Horizontal, symbol Connector:Screw_Terminal_01x02
- removed JP1, JP2: SolderJumper_2_Bridged, symbol Jumper:SolderJumper_2_Bridged
- removed Q12, Q3, Q6, Q9: NMOS, symbol Simulation_SPICE:NMOS
- added C6, C7: C_Polarized_Small, symbol Device:C_Polarized_Small
- added D1: D, symbol Device:D
- added J8: Screw_Terminal_01x03, TerminalBlock_Phoenix:TerminalBlock_Phoenix_MPT-0,5-3-2.54_1x03_P2.54mm_Horizontal, symbol Connector:Screw_Terminal_01x03
- added JP1, JP2: SolderJumper_3_Bridged12, Jumper:SolderJumper-3_P1.3mm_Bridged12_RoundedPad1.0x1.5mm, symbol Jumper:SolderJumper_3_Bridged12
- added Q13, Q3, Q6, Q9: AO3400A, Package_TO_SOT_SMD:SOT-23, symbol Transistor_FET:AO3400A
- SW1: footprint (none) -> Button_Switch_THT:SW_PUSH_6mm_H5mm
- U2: footprint RF_Module:ESP32-WROOM-32 -> Library_Pia:ESP32-Wroom-32
Connections:
- net +24V: now also J6.1 (Pin_1), C6.1, D1.1 (K)
- net GND: now also C6.2, C7.1, J8.2 (Pin_2), Q13.2 (S), Q3.2 (S), Q6.2 (S), Q9.2 (S)
- net RX: now also JP1.3 (B), JP2.1 (A)
- net TX: now also JP1.1 (A), JP2.3 (B)
- net at R21.1, R22.2: now also Q9.1 (G)
- net CW2: now reaches J6.2 (Pin_2)
- net CW2: now also Q6.3 (D)
- net WW2: now reaches J6.3 (Pin_3)
- net WW2: now also Q9.3 (D)
- net WW1: now reaches J5.3 (Pin_3)
- net WW1: now also Q3.3 (D)
- net at R11.1, R12.2: now also Q3.1 (G)
- net CW1: now reaches J5.2 (Pin_2)
- net CW1: now also Q13.3 (D)
- net +5V: now reaches C2.1, U3.3 (VI)
- net +5V: now also C7.2, J8.1 (Pin_1)
- net at R6.1, R7.2: now also Q13.1 (G)
- net at R16.1, R17.2: now also Q6.1 (G)
- net at J3.3 (Pin_3): now also JP2.2 (C)
- net at J3.2 (Pin_2): now also JP1.2 (C)
- new net: D1.2 (A), J8.3 (Pin_3)
Other:
- moved on the sheet: C1, C2, C3, C4, C5, J3, R1, R2, R23, R24, R25, SW1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

Commit message: add more parts
Parts:
- added C8, C9: 10.000uF, Capacitor_THT:CP_Axial_L38.0mm_D18.0mm_P44.00mm_Horizontal, symbol Device:C_Polarized_Small
- added FID1, FID2, FID3: Fiducial, Fiducial:Fiducial_1.5mm_Mask3mm, symbol Mechanical:Fiducial
- added H1, H2, H3, H4: MountingHole, MountingHole:MountingHole_3.2mm_M3, symbol Mechanical:MountingHole
- C6, C7: value C_Polarized_Small -> 470u; footprint (none) -> Capacitor_SMD:CP_Elec_10x10
- D1: footprint (none) -> Package_TO_SOT_THT:TO-220-2_Horizontal_TabDown
Connections:
- net +24V: now also C8.1
- net +3V3: no longer J2.1 (Pin_1), J4.1 (Pin_1), J7.1 (Pin_1)
- net +5V: now also C7.1, J2.1 (Pin_1), J4.1 (Pin_1), J7.1 (Pin_1), J8.3 (Pin_3), C9.1; no longer C7.2, J8.1 (Pin_1)
- net GND: now also C7.2, C8.2, C9.2; no longer C7.1
- net V_IN: now reaches D1.2 (A)
- net V_IN: now also J8.1 (Pin_1); no longer J8.3 (Pin_3)
Other:
- moved on the sheet: C1, C2, C6, C7, D1, J3, J8, JP1, JP2, U3

Commit message: add more tracks
Parts:
- added NT1: NetTie_2, NetTie:NetTie-2_SMD_Pad2.0mm, symbol Device:NetTie_2
- added NT2: NetTie_2, NetTie:NetTie-2_THT_Pad1.0mm, symbol Device:NetTie_2
- SW1: value Reset -> Boot
Connections:
- net LED1: now also U2.37 (IO23); no longer U2.36 (IO22)
- net LED2: now also U2.36 (IO22); no longer U2.37 (IO23)
- removed net GND: C1.2, C2.2, C3.2, C4.2, C5.2, C6.2, C7.2, C8.2, C9.2, J2.3 (Pin_3), J3.6 (Pin_6), J4.3 (Pin_3), J7.3 (Pin_3), J8.2 (Pin_2), Q11.3 (E), Q13.2 (S), Q2.3 (E), Q3.2 (S), Q5.3 (E), Q6.2 (S), Q8.3 (E), Q9.2 (S), R1.2, R12.1, R17.1, R22.1, R23.2, R25.2, R7.1, U2.1 (GND), U2.15 (GND), U2.38 (GND), U2.39 (GND), U3.1 (GND)
- new net GND1: C6.2, C8.2, J8.2 (Pin_2), NT1.1, Q11.3 (E), Q13.2 (S), Q2.3 (E), Q3.2 (S), Q5.3 (E), Q6.2 (S), Q8.3 (E), Q9.2 (S), R12.1, R17.1, R22.1, R7.1
- new net GND2: C2.2, C7.2, C9.2, J2.3 (Pin_3), J4.3 (Pin_3), J7.3 (Pin_3), NT1.2, NT2.1, U3.1 (GND)
- new net GND3: C1.2, C3.2, C4.2, C5.2, J3.6 (Pin_6), NT2.2, R1.2, R23.2, R25.2, U2.1 (GND), U2.15 (GND), U2.38 (GND), U2.39 (GND)
Other:
- moved on the sheet: C6, C7, C8, C9
