File: StreamLite.kicad_pcb (KiCad board)
At the start: 2 copper layers, 78.5 x 48.5 mm, 60 parts, among them J2 Screw_Terminal_01x03, J3 Conn_01x06_Socket, J4 Screw_Terminal_01x03, J5 Screw_Terminal_01x03, J6 Screw_Terminal_01x03, J7 Screw_Terminal_01x03, J8 Screw_Terminal_01x03, Q1 BC327, Q10 BC327, Q11 BC337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

Commit message: add more parts
Parts:
- added C6: 470u, Capacitor_SMD:CP_Elec_10x10, F.Cu at (99.2, 135.9)
- added C7: 470u, Capacitor_SMD:CP_Elec_10x10, F.Cu at (65.2, 146.1)
- added C8: 10.000uF, Capacitor_THT:CP_Axial_L38.0mm_D18.0mm_P44.00mm_Horizontal, F.Cu at (114.5, 139.4)
- added C9: 10.000uF, Capacitor_THT:CP_Axial_L38.0mm_D18.0mm_P44.00mm_Horizontal, F.Cu at (84.3, 95.8)
- added D1: D, Package_TO_SOT_THT:TO-220-2_Horizontal_TabDown, F.Cu at (133.9, 108.7)
- added FID1: Fiducial, Fiducial:Fiducial_1.5mm_Mask3mm, F.Cu at (135.6, 168.8)
- added FID2: Fiducial, Fiducial:Fiducial_1.5mm_Mask3mm, F.Cu at (48.1, 92.8)
- added FID3: Fiducial, Fiducial:Fiducial_1.5mm_Mask3mm, F.Cu at (136.2, 100.1)
- added H1: MountingHole, MountingHole:MountingHole_3.2mm_M3, F.Cu at (43.5, 175.2)
- added H2: MountingHole, MountingHole:MountingHole_3.2mm_M3, F.Cu at (134.2, 95.0)
- added H3: MountingHole, MountingHole:MountingHole_3.2mm_M3, F.Cu at (135.3, 175.8)
- added H4: MountingHole, MountingHole:MountingHole_3.2mm_M3, F.Cu at (42.7, 94.5)
- added kibuzzard-670D99B4: G***, kibuzzard-670D99B4, F.Cu at (105.1, 169.1)
- added kibuzzard-670EF22D: G***, kibuzzard-670EF22D, F.Cu at (88.1, 168.8)
- added kibuzzard-670EF237: G***, kibuzzard-670EF237, F.Cu at (71.0, 168.9)
- added kibuzzard-670EF243: G***, kibuzzard-670EF243, F.Cu at (54.3, 168.8)
- moved J2 132.1 mm to (51.5, 173.7), turned to 0 degrees
- moved kibuzzard-670D983B 131.1 mm to (54.1, 178.1)
- moved J4 130.7 mm to (68.5, 173.7), turned to 0 degrees
- moved kibuzzard-670D9849 129.9 mm to (71.5, 178.1)
- moved J7 129.7 mm to (85.5, 173.7), turned to 0 degrees
- moved kibuzzard-670D9857 129.2 mm to (88.8, 178.1)
- moved kibuzzard-670D97D1 129.2 mm to (122.0, 178.0)
- moved J5 129.2 mm to (102.4, 173.7), turned to 0 degrees
- moved J6 129.1 mm to (119.4, 173.8), turned to 0 degrees
- moved kibuzzard-670D998F 129.0 mm to (105.6, 178.1)
- moved kibuzzard-670D99B4 118.0 mm to (122.0, 168.9)
- moved Q9 109.3 mm to (134.7, 161.9), turned to 0 degrees
- moved Q3 107.9 mm to (104.0, 162.1), turned to 0 degrees
- moved R22 104.8 mm to (130.5, 161.8), turned to 90 degrees
- moved Q6 103.9 mm to (119.8, 162.3), turned to 0 degrees
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Connections:
- J2 pad 1: +3V3 -> +5V
- J4 pad 1: +3V3 -> +5V
- J7 pad 1: +3V3 -> +5V
- J8 pad 1: +5V -> /V_IN
- J8 pad 3: +24V -> +5V
Routing:
- net GND: track 57.4 -> 173.0 mm
- net +5V: track 38.8 -> 146.7 mm, vias 0 -> 1
- net +24V: track 77.9 -> 167.1 mm, vias 0 -> 2
- net CCT1_WW: track 0.00 -> 66.9 mm, vias 0 -> 1
- net /V_IN: track 0.00 -> 39.8 mm
- net /CW1: track 0.00 -> 22.8 mm, vias 0 -> 1
- net /WW2: track 0.00 -> 22.7 mm, vias 0 -> 1
- net Net-(Q1-B): track 0.00 -> 14.6 mm
- net /WW1: track 0.00 -> 12.5 mm, vias 0 -> 1
- net /CW2: track 0.00 -> 11.7 mm, vias 0 -> 1
- net Net-(Q7-B): track 0.00 -> 11.5 mm
- net Net-(Q10-B): track 0.00 -> 10.3 mm
- net Net-(Q6-G): track 0.00 -> 7.94 mm
- net Net-(Q9-G): track 0.00 -> 7.83 mm
- net Net-(U2-EN): track 7.66 -> 0.00 mm
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- added copper zone on F.Cu, net +24V
- added copper zone on B.Cu, net GND
- added copper zone on F.Cu, net GND
Other:
- board size 78.5 x 48.5 mm -> 98.8 x 88.5 mm

Commit message: add more tracks
Parts:
- added NT1: NetTie_2, NetTie:NetTie-2_SMD_Pad2.0mm, F.Cu at (89.4, 144.5)
- added NT2: NetTie_2, NetTie:NetTie-2_THT_Pad1.0mm, B.Cu at (47.3, 144.4)
- SW1: value Reset -> Boot
- moved U3 15.9 mm to (51.5, 143.4), turned to 90 degrees
- moved C2 14.6 mm to (51.7, 149.5), turned to 180 degrees
- moved C1 11.0 mm to (49.8, 138.0), turned to 180 degrees
- moved FID1 10.3 mm to (130.2, 177.6)
- moved R1 7.73 mm to (50.4, 101.1), turned to -90 degrees
- moved R25 4.32 mm to (67.9, 109.1), turned to 90 degrees
- moved C8 3.44 mm to (114.6, 142.8)
- moved C9 2.59 mm to (84.3, 98.3)
- moved C7 1.29 mm to (66.5, 145.9), turned to -90 degrees
- moved JP2 1.13 mm to (52.0, 104.8)
- moved JP1 0.90 mm to (52.1, 108.1)
- moved J3 0.49 mm to (53.8, 101.4)
Connections:
- C1 pad 2: GND -> GND3
- C2 pad 2: GND -> GND2
- C3 pad 2: GND -> GND3
- C4 pad 2: GND -> GND3
- C5 pad 2: GND -> GND3
- C6 pad 2: GND -> GND1
- C7 pad 2: GND -> GND2
- C8 pad 2: GND -> GND1
- C9 pad 2: GND -> GND2
- J2 pad 3: GND -> GND2
- J3 pad 6: GND -> GND3
- J4 pad 3: GND -> GND2
- J7 pad 3: GND -> GND2
- J8 pad 2: GND -> GND1
- Q11 pad 3: GND -> GND1
- Q13 pad 2: GND -> GND1
- Q2 pad 3: GND -> GND1
- Q3 pad 2: GND -> GND1
- Q5 pad 3: GND -> GND1
- Q6 pad 2: GND -> GND1
- Q8 pad 3: GND -> GND1
- Q9 pad 2: GND -> GND1
- R1 pad 2: GND -> GND3
- R12 pad 1: GND -> GND1
- R17 pad 1: GND -> GND1
- R22 pad 1: GND -> GND1
- R23 pad 2: GND -> GND3
- R25 pad 2: GND -> GND3
- R7 pad 1: GND -> GND1
- U2 pad 1: GND -> GND3
- U2 pad 15: GND -> GND3
- U2 pad 36: LED1 -> LED2
- U2 pad 37: LED2 -> LED1
- U2 pad 38: GND -> GND3
- U2 pad 39: GND -> GND3
- U3 pad 1: GND -> GND2
Routing:
- net GND1: track 0.00 -> 183.8 mm, vias 0 -> 7
- net GND: track 173.0 -> 0.00 mm, vias 2 -> 0
- net GND2: track 0.00 -> 127.4 mm, vias 0 -> 8
- net GND3: track 0.00 -> 103.8 mm, vias 0 -> 1
- net LED2: track 0.00 -> 79.2 mm, vias 0 -> 1
- net +3V3: track 25.7 -> 99.2 mm, vias 0 -> 2
- net LED1: track 0.00 -> 73.1 mm, vias 0 -> 1
- net CCT1_CW: track 0.00 -> 62.8 mm, vias 0 -> 2
- net LED3: track 0.00 -> 60.5 mm, vias 0 -> 1
- net CCT2_WW: track 0.00 -> 56.0 mm, vias 0 -> 2
- net CCT2_CW: track 0.00 -> 39.9 mm, vias 0 -> 2
- net Net-(U2-IO0): track 0.00 -> 34.0 mm, vias 0 -> 2
- net +5V: track 146.7 -> 173.3 mm, vias 1 -> 4
- net +24V: track 167.1 -> 186.1 mm, vias 2 -> 3
- net Net-(R1-Pad1): track 0.00 -> 13.2 mm, vias 0 -> 1
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- added copper zone on F.Cu, net +5V
- added copper zone on B.Cu, net GND1
- added copper zone on B.Cu, net GND3
- added copper zone on F.Cu, net GND3
- removed copper zone on F.Cu, net +24V
- removed copper zone on B.Cu, net GND
- removed copper zone on F.Cu, net GND

Commit message: add schematic
Parts:
- removed kibuzzard-670EF22D: G***, kibuzzard-670EF22D
- added C10: 100n, Capacitor_SMD:C_0805_2012Metric_Pad1.18x1.45mm_HandSolder, F.Cu at (51.5, 157.3)
- added G***: LOGO, Library_Pia:Logo-kuh, F.Cu at (132.7, 143.0)
- added Q12: D4185, Library_Pia:TO-252-3_TabPin2_D4185, F.Cu at (58.7, 156.2)
- added Q14: BC547, Package_TO_SOT_THT:TO-92_Inline, F.Cu at (57.0, 141.7)
- added R26: 1k, Capacitor_SMD:C_1206_3216Metric_Pad1.33x1.80mm_HandSolder, F.Cu at (42.0, 165.5)
- added R27: 1k, Capacitor_SMD:C_1206_3216Metric_Pad1.33x1.80mm_HandSolder, F.Cu at (44.4, 165.5)
- added R28: 1k, Capacitor_SMD:C_1206_3216Metric_Pad1.33x1.80mm_HandSolder, F.Cu at (46.8, 165.5)
- added R29: 2k2, Capacitor_SMD:C_1206_3216Metric_Pad1.33x1.80mm_HandSolder, F.Cu at (56.5, 146.3)
- added R30: 1k, Capacitor_SMD:C_1206_3216Metric_Pad1.33x1.80mm_HandSolder, F.Cu at (59.8, 106.1)
- added U1: 4049, Package_SO:SO-16_3.9x9.9mm_P1.27mm, F.Cu at (45.1, 157.0)
- added kibuzzard-672436BF: G***, kibuzzard-672436BF, F.Cu at (88.6, 169.4)
- added kibuzzard-67243969: G***, kibuzzard-67243969, F.Cu at (95.3, 106.2)
- added kibuzzard-67243A60: G***, kibuzzard-67243A60, F.Cu at (114.6, 146.7)
- added kibuzzard-67243A6C: G***, kibuzzard-67243A6C, F.Cu at (114.6, 143.5)
- C8, C9: footprint Capacitor_THT:CP_Axial_L38.0mm_D18.0mm_P44.00mm_Horizontal -> Library_Pia:Capacitor_L38.0mm_D18.0mm_P10_Horizontal
- J8: footprint TerminalBlock_Phoenix:TerminalBlock_Phoenix_MPT-0,5-3-2.54_1x03_P2.54mm_Horizontal -> TerminalBlock_MetzConnect:TerminalBlock_MetzConnect_Type701_RT11L03HGLU_1x03_P6.35mm_Horizontal
- moved C8 31.4 mm to (120.5, 112.1)
- moved D1 25.6 mm to (108.5, 106.3)
- moved C9 19.7 mm to (79.4, 117.5), turned to 90 degrees
- moved J8 8.99 mm to (93.8, 96.5), turned to 0 degrees
- moved NT1 4.65 mm to (90.8, 140.0)
- moved kibuzzard-670EF237 0.79 mm to (71.0, 169.7)
- moved kibuzzard-670EF243 0.79 mm to (54.4, 169.6)
- moved C4 0.42 mm to (47.6, 133.5)
- moved C3 0.40 mm to (47.6, 131.5)
- moved SW1 0.26 mm to (41.0, 100.3)
- moved R2 0.14 mm to (52.0, 133.4)
Connections:
- J2 pad 1: +5V -> +5VP
- J2 pad 2: LED1 -> Net-(J2-Pin_2)
- J4 pad 1: +5V -> +5VP
- J4 pad 2: LED2 -> Net-(J4-Pin_2)
- J7 pad 1: +5V -> +5VP
- J7 pad 2: LED3 -> Net-(J7-Pin_2)
- J8 pad 1: /V_IN -> +5V
- J8 pad 3: +5V -> /V_IN
- U2 pad 33: unconnected-(U2-IO21-Pad33) -> Sig_5V_Off
Routing:
- net +5VP: track 0.00 -> 80.7 mm, vias 0 -> 4
- net GND2: track 127.4 -> 193.5 mm, vias 8 -> 21
- net +5V: track 173.3 -> 115.0 mm, vias 4 -> 5
- net Net-(J7-Pin_2): track 0.00 -> 46.4 mm, vias 0 -> 1
- net Net-(Q14-B): track 0.00 -> 42.1 mm, vias 0 -> 1
- net GND1: track 183.8 -> 222.7 mm, vias 7 -> 11
- net Net-(J4-Pin_2): track 0.00 -> 32.4 mm, vias 0 -> 1
- net /V_IN: track 39.8 -> 11.2 mm
- net LED3: track 60.5 -> 34.8 mm, vias 1 -> 2
- net LED2: track 79.2 -> 55.9 mm, vias 1 -> 2
- net Net-(U1-Pad4): track 0.00 -> 22.2 mm, vias 0 -> 2
- net LED1: track 73.1 -> 51.6 mm, vias 1 -> 2
- net Net-(U1-Pad11): track 0.00 -> 19.4 mm, vias 0 -> 2
- net Net-(Q12-G): track 0.00 -> 19.2 mm, vias 0 -> 2
- net Net-(U1-Pad14): track 0.00 -> 18.0 mm, vias 0 -> 2
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- added copper zone on B.Cu, net +24V
- added copper zone on B.Cu, net +5V
- added copper zone on F.Cu, net GND1
- added copper zone on B.Cu, net GND2
